Commit message: Add lidar, caster wheel, SLAM mapping, Nav2 autonomous navigation

File: atlas_monitor/urdf/robot.urdf (robot description, URDF)
Before this commit: robot atlas_bot, 3 links, 2 joints
Links:
- added link caster_wheel, mass 0.1; collision sphere radius=0.05; visual sphere radius=0.05
- added link lidar_link, mass 0.1; collision cylinder length=0.04 radius=0.05; visual cylinder length=0.04 radius=0.05
Joints:
- added joint caster_joint: type fixed, parent base_link, child caster_wheel, origin xyz=0.2 0 -0.05 rpy=0 0 0
- added joint lidar_joint: type fixed, parent base_link, child lidar_link, origin xyz=0 0 0.13 rpy=0 0 0
